File: fusilera 24 canales.kicad_pcb (KiCad board)
At the start: 4 copper layers, 202 parts, among them J1 +12V borne M6, J2 GND borne M5, Q1 MMBT2222A, Q101 MMBT2222A, Q102 MMBT2222A, Q103 MMBT2222A, Q104 MMBT2222A, Q105 MMBT2222A, Q106 MMBT2222A, Q107 MMBT2222A, Q108 MMBT2222A, Q2 MMBT2222A, Q3 MMBT2222A, Q4 MMBT2222A, Q5 MMBT2222A, Q6 MMBT2222A, Q7 MMBT2222A, Q8 MMBT2222A, U1 LM339D, U10 BTS50010-1TAD, U101 LM339D, U102 74HC132D, U103 BTS50010-1TAD, U108 BTS50010-1TAD, U109 74HC132D, U11 BTS50010-1TAD, U110 BTS50010-1TAD, U111 BTS50010-1TAD, U2 74HC132D, U3 BTS50010-1TAD, U4 MCP23017-E/SO, U5 MCP23017-E/SO, U6 LM5164DDA, U7 AP2112K-3.3, U8 BTS50010-1TAD, U9 74HC132D

Commit message: Añade la Celda3, gira los canales 3 y 4 y rutea los grupos movidos de la Celda1
Agrega la tercera instancia de la celda al esquemático (referencias +200) y
pasa sus footprints al PCB. En la Celda1 los canales 3 y 4 quedan girados 180°
al lado izquierdo con la lógica compartida en el centro, y se rutean con un
enrutador de rejilla propio IS3, IS4, FALLA3, FALLA4, los umbrales y los
pull-ups de los comparadores, más las vías de plano de C18, C19, R31 y R32.
Se documenta la decisión de arquitectura y el riesgo del bus hacia el
controlador en CONTEXTO_PROYECTO.md.
Parts:
- added C201: 100uF 16V, Capacitor_SMD:CP_Elec_6.3x5.4, F.Cu at (215.9, 76.8)
- added C202: 100nF, Capacitor_SMD:C_0805_2012Metric, F.Cu at (245.8, 58.1)
- added C203: 1uF 25V, Capacitor_SMD:CP_Elec_4x5.4, F.Cu at (214.5, 30.2)
- added C204: 100nF, Capacitor_SMD:C_0805_2012Metric, F.Cu at (245.8, 61.1)
- added C205: 1uF 25V, Capacitor_SMD:CP_Elec_4x5.4, F.Cu at (214.5, 36.1)
- added C216: 1uF 25V, Capacitor_SMD:CP_Elec_4x5.4, F.Cu at (214.5, 41.9)
- added C217: 1uF 25V, Capacitor_SMD:CP_Elec_4x5.4, F.Cu at (214.5, 47.8)
- added C218: 1uF 25V, Capacitor_SMD:CP_Elec_4x5.4, F.Cu at (214.5, 53.6)
- added C219: 1uF 25V, Capacitor_SMD:CP_Elec_4x5.4, F.Cu at (222.2, 30.2)
- added C220: 100nF, Capacitor_SMD:C_0805_2012Metric, F.Cu at (245.8, 64.1)
- added C221: 1uF 25V, Capacitor_SMD:CP_Elec_4x5.4, F.Cu at (222.2, 36.1)
- added C222: 1uF 25V, Capacitor_SMD:CP_Elec_4x5.4, F.Cu at (222.2, 41.9)
- added D201: BAT54C, Package_TO_SOT_SMD:SOT-23, F.Cu at (226.4, 58.8)
- added D202: LED verde, LED_SMD:LED_0805_2012Metric, F.Cu at (250.4, 28.8)
- added D203: LED rojo, LED_SMD:LED_0805_2012Metric, F.Cu at (250.4, 31.9)
- added D207: LED verde, LED_SMD:LED_0805_2012Metric, F.Cu at (250.4, 34.9)
- added D208: BAT54C, Package_TO_SOT_SMD:SOT-23, F.Cu at (226.4, 63.2)
- added D209: LED rojo, LED_SMD:LED_0805_2012Metric, F.Cu at (250.4, 37.9)
- added D210: LED rojo, LED_SMD:LED_0805_2012Metric, F.Cu at (250.4, 41.0)
- added D211: LED rojo, LED_SMD:LED_0805_2012Metric, F.Cu at (250.4, 44.0)
- added D212: LED verde, LED_SMD:LED_0805_2012Metric, F.Cu at (250.4, 47.1)
- added D213: LED verde, LED_SMD:LED_0805_2012Metric, F.Cu at (250.4, 50.1)
- added D214: BAT54C, Package_TO_SOT_SMD:SOT-23, F.Cu at (226.4, 67.7)
- added D215: BAT54C, Package_TO_SOT_SMD:SOT-23, F.Cu at (231.3, 58.8)
- added Q201: MMBT2222A, Package_TO_SOT_SMD:SOT-23, F.Cu at (231.3, 63.2)
- added Q202: MMBT2222A, Package_TO_SOT_SMD:SOT-23, F.Cu at (231.3, 67.7)
- added Q203: MMBT2222A, Package_TO_SOT_SMD:SOT-23, F.Cu at (236.2, 58.8)
- added Q204: MMBT2222A, Package_TO_SOT_SMD:SOT-23, F.Cu at (236.2, 63.2)
- added Q205: MMBT2222A, Package_TO_SOT_SMD:SOT-23, F.Cu at (236.2, 67.7)
- added Q206: MMBT2222A, Package_TO_SOT_SMD:SOT-23, F.Cu at (241.1, 58.8)
- added Q207: MMBT2222A, Package_TO_SOT_SMD:SOT-23, F.Cu at (241.1, 63.2)
- added Q208: MMBT2222A, Package_TO_SOT_SMD:SOT-23, F.Cu at (241.1, 67.7)
- added R201: umbral, Resistor_THT:R_Axial_DIN0207_L6.3mm_D2.5mm_P10.16mm_Horizontal, F.Cu at (212.2, 58.6)
- added R202: 10k, Resistor_SMD:R_0805_2012Metric, F.Cu at (228.3, 28.8)
- added R203: 10k, Resistor_SMD:R_0805_2012Metric, F.Cu at (228.3, 31.7)
- added R204: 4.7k, Resistor_SMD:R_0805_2012Metric, F.Cu at (228.3, 34.7)
- added R205: 4.7k, Resistor_SMD:R_0805_2012Metric, F.Cu at (228.3, 37.6)
- added R206: 10k, Resistor_SMD:R_0805_2012Metric, F.Cu at (228.3, 40.6)
- added R207: 100k, Resistor_SMD:R_0805_2012Metric, F.Cu at (228.3, 43.5)
- added R208: 100k, Resistor_SMD:R_0805_2012Metric, F.Cu at (228.3, 46.5)
- added R209: 1k, Resistor_SMD:R_0805_2012Metric, F.Cu at (228.3, 49.4)
- added R210: 2.2k, Resistor_SMD:R_0805_2012Metric, F.Cu at (228.3, 52.4)
- added R211: 4.7k, Resistor_SMD:R_0805_2012Metric, F.Cu at (232.7, 28.8)
- added R212: 1k, Resistor_SMD:R_0805_2012Metric, F.Cu at (232.7, 31.7)
- added R219: 4.7k, Resistor_SMD:R_0805_2012Metric, F.Cu at (232.7, 34.7)
- added R220: 4.7k, Resistor_SMD:R_0805_2012Metric, F.Cu at (232.7, 37.6)
- added R221: 2.2k, Resistor_SMD:R_0805_2012Metric, F.Cu at (232.7, 40.6)
- added R222: 100k, Resistor_SMD:R_0805_2012Metric, F.Cu at (232.7, 43.5)
- added R223: 100k, Resistor_SMD:R_0805_2012Metric, F.Cu at (232.7, 46.5)
- added R224: 1k, Resistor_SMD:R_0805_2012Metric, F.Cu at (232.7, 49.4)
- added R225: 1k, Resistor_SMD:R_0805_2012Metric, F.Cu at (232.7, 52.4)
- added R226: 4.7k, Resistor_SMD:R_0805_2012Metric, F.Cu at (237.1, 28.8)
- added R227: 10k, Resistor_SMD:R_0805_2012Metric, F.Cu at (237.1, 31.7)
- added R228: 10k, Resistor_SMD:R_0805_2012Metric, F.Cu at (237.1, 34.7)
- added R229: umbral, Resistor_THT:R_Axial_DIN0207_L6.3mm_D2.5mm_P10.16mm_Horizontal, F.Cu at (212.2, 62.6)
- added R230: 10k, Resistor_SMD:R_0805_2012Metric, F.Cu at (237.1, 37.6)
- added R231: 10k, Resistor_SMD:R_0805_2012Metric, F.Cu at (237.1, 40.6)
- added R232: 10k, Resistor_SMD:R_0805_2012Metric, F.Cu at (237.1, 43.5)
- added R233: 1k, Resistor_SMD:R_0805_2012Metric, F.Cu at (237.1, 46.5)
- added R234: 1k, Resistor_SMD:R_0805_2012Metric, F.Cu at (237.1, 49.4)
- added R235: 4.7k, Resistor_SMD:R_0805_2012Metric, F.Cu at (237.1, 52.4)
- added R236: 4.7k, Resistor_SMD:R_0805_2012Metric, F.Cu at (241.5, 28.8)
- added R237: 4.7k, Resistor_SMD:R_0805_2012Metric, F.Cu at (241.5, 31.7)
- added R238: 4.7k, Resistor_SMD:R_0805_2012Metric, F.Cu at (241.5, 34.7)
- added R239: 4.7k, Resistor_SMD:R_0805_2012Metric, F.Cu at (241.5, 37.6)
- added R240: 4.7k, Resistor_SMD:R_0805_2012Metric, F.Cu at (241.5, 40.6)
- added R241: 2.2k, Resistor_SMD:R_0805_2012Metric, F.Cu at (241.5, 43.5)
- added R242: 2.2k, Resistor_SMD:R_0805_2012Metric, F.Cu at (241.5, 46.5)
- added R243: 100k, Resistor_SMD:R_0805_2012Metric, F.Cu at (241.5, 49.4)
- added R244: 100k, Resistor_SMD:R_0805_2012Metric, F.Cu at (241.5, 52.4)
- added R245: 100k, Resistor_SMD:R_0805_2012Metric, F.Cu at (245.9, 28.8)
- added R246: 100k, Resistor_SMD:R_0805_2012Metric, F.Cu at (245.9, 31.7)
- added R247: 1k, Resistor_SMD:R_0805_2012Metric, F.Cu at (245.9, 34.7)
- added R248: 1k, Resistor_SMD:R_0805_2012Metric, F.Cu at (245.9, 37.6)
- added R249: umbral, Resistor_THT:R_Axial_DIN0207_L6.3mm_D2.5mm_P10.16mm_Horizontal, F.Cu at (212.2, 66.7)
- added R250: 10k, Resistor_SMD:R_0805_2012Metric, F.Cu at (245.9, 40.6)
- added R251: umbral, Resistor_THT:R_Axial_DIN0207_L6.3mm_D2.5mm_P10.16mm_Horizontal, F.Cu at (212.2, 70.7)
- added R252: 10k, Resistor_SMD:R_0805_2012Metric, F.Cu at (245.9, 43.5)
- added R253: 10k, Resistor_SMD:R_0805_2012Metric, F.Cu at (245.9, 46.5)
- added R254: 10k, Resistor_SMD:R_0805_2012Metric, F.Cu at (245.9, 49.4)
- added U201: LM339D, Package_SO:SOIC-14_3.9x8.7mm_P1.27mm, F.Cu at (228.1, 75.2)
- added U202: 74HC132D, Package_SO:SOIC-14_3.9x8.7mm_P1.27mm, F.Cu at (236.6, 75.2)
- added U203: BTS50010-1TAD, Package_TO_SOT_SMD:TO-263-7_TabPin4, F.Cu at (203.6, 33.5)
- added U208: BTS50010-1TAD, Package_TO_SOT_SMD:TO-263-7_TabPin4, F.Cu at (203.6, 45.8)
- added U209: 74HC132D, Package_SO:SOIC-14_3.9x8.7mm_P1.27mm, F.Cu at (245.0, 75.2)
- added U210: BTS50010-1TAD, Package_TO_SOT_SMD:TO-263-7_TabPin4, F.Cu at (203.6, 58.2)
- added U211: BTS50010-1TAD, Package_TO_SOT_SMD:TO-263-7_TabPin4, F.Cu at (203.6, 70.5)
- moved C6 227.3 mm to (-2.35, 122.0)
- moved U5 132.0 mm to (-18.6, 111.5)
- moved U4 121.3 mm to (119.3, 197.6)
- moved C116 120.0 mm to (45.9, 259.1)
- moved D101 120.0 mm to (56.4, 278.0)
- moved D103 120.0 mm to (48.9, 280.8)
- moved D107 120.0 mm to (49.6, 264.9)
- moved D108 120.0 mm to (57.3, 259.9)
- moved D109 120.0 mm to (49.6, 262.6)
- moved Q103 120.0 mm to (57.3, 264.9)
- moved R104 120.0 mm to (60.1, 277.3)
- moved R105 120.0 mm to (60.1, 279.3)
- moved R108 120.0 mm to (53.4, 276.5)
- moved R110 120.0 mm to (52.6, 283.0)
- moved R112 120.0 mm to (52.4, 280.8)
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Routing:
- net Net-(U11-IS): track 107.0 -> 75.6 mm
- net /Celda1/FALLA4: track 30.5 -> 57.6 mm
- net Net-(R53-Pad1): track 56.7 -> 39.4 mm, vias 2 -> 4
- net Net-(U1B-+): track 16.6 -> 31.4 mm
- net Net-(U1C-+): track 13.5 -> 26.7 mm, vias 2 -> 1
- net Net-(U1D-+): track 13.8 -> 27.0 mm, vias 0 -> 1
- net Net-(R54-Pad1): track 44.9 -> 32.9 mm
- net +3.3V: track 143.2 -> 131.5 mm, vias 36 -> 37
- net /Celda1/FALLA3: track 30.9 -> 35.9 mm
- net Net-(U1A-+): track 12.0 -> 8.89 mm
- net GND: track 198.6 -> 195.9 mm
- net Net-(U10-IS): track 95.8 -> 95.3 mm, vias 6 -> 7

Commit message: Conecta las celdas con el micro, dibuja el contorno y reubica los bloques
Cablea en el esquemático raíz las salidas ESP32_OUT y las entradas FALLA de las
tres celdas a pines de la ESP32 (A1) y del MCP23017 (U4) mediante etiquetas
locales, de modo que el PCB muestra el ratsnest hacia el controlador. Dibuja el
contorno de la placa en Edge.Cuts (123 x 191 mm), ajusta los planos de GND y
+3,3 V a ese contorno y reubica las celdas, el controlador y el bloque de poder.
Se registra la hoja Celda3 en el proyecto y se actualiza CONTEXTO_PROYECTO.md.
Parts:
- moved D210 417.4 mm to (-140.4, 187.7)
- moved D212 416.1 mm to (-140.4, 189.9), turned to 180 degrees
- moved R247 414.2 mm to (-140.5, 183.5), turned to 90 degrees
- moved D211 410.9 mm to (-140.8, 170.0)
- moved D213 409.8 mm to (-140.8, 172.3), turned to 180 degrees
- moved R248 406.6 mm to (-140.3, 164.6), turned to 90 degrees
- moved R241 405.8 mm to (-136.9, 189.9), turned to 180 degrees
- moved R246 403.8 mm to (-135.3, 164.8), turned to 90 degrees
- moved R245 402.0 mm to (-129.3, 173.0)
- moved R237 400.7 mm to (-129.2, 183.9), turned to 180 degrees
- moved R238 400.4 mm to (-129.2, 185.9)
- moved R244 400.0 mm to (-136.4, 183.5), turned to 90 degrees
- moved R233 399.8 mm to (-136.9, 187.7), turned to 180 degrees
- moved R242 399.0 mm to (-137.1, 172.3), turned to 180 degrees
- moved R243 396.4 mm to (-128.9, 190.4)
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Connections:
- A1 pad 10: unconnected-(A1-D27-Pad10) -> /D27
- A1 pad 11: unconnected-(A1-D14-Pad11) -> /D14
- A1 pad 13: unconnected-(A1-D13-Pad13) -> /D13
- A1 pad 16: unconnected-(A1-D23-Pad16) -> /D23
- A1 pad 2: unconnected-(A1-VP/GPIO36-Pad2) -> /VP
- A1 pad 21: unconnected-(A1-D19-Pad21) -> /D19
- A1 pad 22: unconnected-(A1-D18-Pad22) -> /D18
- A1 pad 24: unconnected-(A1-TX2/GPIO17-Pad24) -> /TX2
- A1 pad 25: unconnected-(A1-RX2/GPIO16-Pad25) -> /RX2
- A1 pad 26: unconnected-(A1-D4-Pad26) -> /D4
- A1 pad 3: unconnected-(A1-VN/GPIO39-Pad3) -> /VN
- A1 pad 4: unconnected-(A1-D34-Pad4) -> /D34
- A1 pad 5: unconnected-(A1-D35-Pad5) -> /D35
- A1 pad 6: unconnected-(A1-D32-Pad6) -> /D32
- A1 pad 7: unconnected-(A1-D33-Pad7) -> /D33
- A1 pad 8: unconnected-(A1-D25-Pad8) -> /D25
- A1 pad 9: unconnected-(A1-D26-Pad9) -> /D26
- R105 pad 2: /Celda2/ESP32_OUT1 -> /D25
- R11 pad 2: /Celda1/FALLA1 -> /RX2
- R111 pad 2: /Celda2/FALLA1 -> /D34
- R112 pad 1: /Celda2/FALLA1 -> /D34
- R12 pad 1: /Celda1/FALLA1 -> /RX2
- R120 pad 2: /Celda2/ESP32_OUT2 -> /D26
- R125 pad 1: /Celda2/FALLA2 -> /D35
- R126 pad 2: /Celda2/FALLA2 -> /D35
- R133 pad 1: /Celda2/FALLA3 -> /D32
- R134 pad 1: /Celda2/FALLA4 -> /D33
- R135 pad 2: /Celda2/FALLA3 -> /D32
- R136 pad 2: /Celda2/FALLA4 -> /D33
- R138 pad 2: /Celda2/ESP32_OUT3 -> /D27
- R140 pad 2: /Celda2/ESP32_OUT4 -> /D14
- R20 pad 2: /Celda1/ESP32_OUT2 -> /D19
- R205 pad 2: /Celda3/ESP32_OUT1 -> /D13
- R211 pad 2: /Celda3/FALLA1 -> /U4-GPA3
- R212 pad 1: /Celda3/FALLA1 -> /U4-GPA3
- R220 pad 2: /Celda3/ESP32_OUT2 -> /U4-GPA0
- R225 pad 1: /Celda3/FALLA2 -> /U4-GPA4
- R226 pad 2: /Celda3/FALLA2 -> /U4-GPA4
- R233 pad 1: /Celda3/FALLA3 -> /U4-GPA5
- R234 pad 1: /Celda3/FALLA4 -> /U4-GPA6
- R235 pad 2: /Celda3/FALLA3 -> /U4-GPA5
- R236 pad 2: /Celda3/FALLA4 -> /U4-GPA6
- R238 pad 2: /Celda3/ESP32_OUT3 -> /U4-GPA1
- R240 pad 2: /Celda3/ESP32_OUT4 -> /U4-GPA2
- R25 pad 1: /Celda1/FALLA2 -> /D4
- R26 pad 2: /Celda1/FALLA2 -> /D4
- R33 pad 1: /Celda1/FALLA3 -> /VP
- R34 pad 1: /Celda1/FALLA4 -> /VN
- R35 pad 2: /Celda1/FALLA3 -> /VP
- R36 pad 2: /Celda1/FALLA4 -> /VN
- R38 pad 2: /Celda1/ESP32_OUT3 -> /D18
- R40 pad 2: /Celda1/ESP32_OUT4 -> /TX2
- R5 pad 2: /Celda1/ESP32_OUT1 -> /D23
- U102 pad 10: /Celda2/FALLA2 -> /D35
- U102 pad 11: /Celda2/FALLA2 -> /D35
- U102 pad 2: /Celda2/FALLA1 -> /D34
- U102 pad 6: /Celda2/FALLA1 -> /D34
- U109 pad 10: /Celda2/FALLA4 -> /D33
- U109 pad 11: /Celda2/FALLA4 -> /D33
- U109 pad 2: /Celda2/FALLA3 -> /D32
- U109 pad 6: /Celda2/FALLA3 -> /D32
- U2 pad 10: /Celda1/FALLA2 -> /D4
- U2 pad 11: /Celda1/FALLA2 -> /D4
- U2 pad 2: /Celda1/FALLA1 -> /RX2
- U2 pad 6: /Celda1/FALLA1 -> /RX2
- U202 pad 10: /Celda3/FALLA2 -> /U4-GPA4
- U202 pad 11: /Celda3/FALLA2 -> /U4-GPA4
- U202 pad 2: /Celda3/FALLA1 -> /U4-GPA3
- U202 pad 6: /Celda3/FALLA1 -> /U4-GPA3
- U209 pad 10: /Celda3/FALLA4 -> /U4-GPA6
- U209 pad 11: /Celda3/FALLA4 -> /U4-GPA6
- U209 pad 2: /Celda3/FALLA3 -> /U4-GPA5
- U209 pad 6: /Celda3/FALLA3 -> /U4-GPA5
- U4 pad 21: unconnected-(U4-GPA0-Pad21) -> /U4-GPA0
- U4 pad 22: unconnected-(U4-GPA1-Pad22) -> /U4-GPA1
- U4 pad 23: unconnected-(U4-GPA2-Pad23) -> /U4-GPA2
- U4 pad 24: unconnected-(U4-GPA3-Pad24) -> /U4-GPA3
- U4 pad 25: unconnected-(U4-GPA4-Pad25) -> /U4-GPA4
- U4 pad 26: unconnected-(U4-GPA5-Pad26) -> /U4-GPA5
- U4 pad 27: unconnected-(U4-GPA6-Pad27) -> /U4-GPA6
- U4 pad 28: unconnected-(U4-GPA7-Pad28) -> /U4-GPA7
- U9 pad 10: /Celda1/FALLA4 -> /VN
- U9 pad 11: /Celda1/FALLA4 -> /VN
- U9 pad 2: /Celda1/FALLA3 -> /VP
- U9 pad 6: /Celda1/FALLA3 -> /VP
Routing:
- net +12V: track 0.00 -> 431.6 mm
- net /U4-GPA6: track 0.00 -> 214.5 mm, vias 0 -> 4
- net /U4-GPA5: track 0.00 -> 203.8 mm, vias 0 -> 3
- net /U4-GPA1: track 0.00 -> 200.2 mm
- net /U4-GPA2: track 0.00 -> 169.8 mm, vias 0 -> 2
- net /U4-GPA3: track 0.00 -> 167.8 mm, vias 0 -> 3
- net /U4-GPA4: track 0.00 -> 160.7 mm, vias 0 -> 4
- net /U4-GPA0: track 0.00 -> 137.7 mm
- net /D23: track 0.00 -> 121.3 mm
- net /D13: track 0.00 -> 119.8 mm, vias 0 -> 1
- net /VN: track 0.00 -> 117.8 mm, vias 0 -> 5
- net /D35: track 0.00 -> 113.1 mm, vias 0 -> 5
- net /RX2: track 0.00 -> 97.5 mm, vias 0 -> 3
- net Net-(U201C--): track 0.00 -> 95.3 mm, vias 0 -> 7
- net /D34: track 0.00 -> 92.8 mm, vias 0 -> 3
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Other:
- board outline added: 123 x 191.1 mm
