File: fusilera 24 canales.kicad_pcb (KiCad board)
At the start: 4 copper layers, 123 x 191.1 mm, 463 parts, among them J1 +12V borne M6, J2 GND borne M5, Q1 MMBT2222A, Q101 MMBT2222A, Q102 MMBT2222A, Q103 MMBT2222A, Q104 MMBT2222A, Q105 MMBT2222A, Q106 MMBT2222A, Q107 MMBT2222A, Q108 MMBT2222A, Q2 MMBT2222A, Q201 MMBT2222A, Q202 MMBT2222A, Q203 MMBT2222A, Q204 MMBT2222A, Q205 MMBT2222A, Q206 MMBT2222A, Q207 MMBT2222A, Q208 MMBT2222A, Q3 MMBT2222A, Q301 MMBT2222A, Q302 MMBT2222A, Q303 MMBT2222A, Q304 MMBT2222A, Q305 MMBT2222A, Q306 MMBT2222A, Q307 MMBT2222A, Q308 MMBT2222A, Q4 MMBT2222A, Q401 MMBT2222A, Q402 MMBT2222A, Q403 MMBT2222A, Q404 MMBT2222A, Q405 MMBT2222A, Q406 MMBT2222A, Q407 MMBT2222A, Q408 MMBT2222A, Q5 MMBT2222A, Q6 MMBT2222A, Q7 MMBT2222A, Q8 MMBT2222A, U1 LM339D, U10 BTS50010-1TAD, U101 LM339D, U102 74HC132D, U103 BTS50010-1TAD, U108 BTS50010-1TAD, U109 74HC132D, U11 BTS50010-1TAD, U110 BTS50010-1TAD, U111 BTS50010-1TAD, U2 74HC132D, U201 LM339D, U202 74HC132D, U203 BTS50010-1TAD, U208 BTS50010-1TAD, U209 74HC132D, U210 BTS50010-1TAD, U211 BTS50010-1TAD, U3 BTS50010-1TAD, U301 LM339D, U302 74HC132D, U303 BTS50010-1TAD, U308 BTS50010-1TAD, U309 74HC132D, U310 BTS50010-1TAD, U311 BTS50010-1TAD, U4 MCP23017-E/SO, U401 LM339D, U402 74HC132D, U403 BTS50010-1TAD, U408 BTS50010-1TAD, U409 74HC132D, U410 BTS50010-1TAD, U411 BTS50010-1TAD, U5 MCP23017-E/SO, U6 LM5164DDA, U7 AP2112K-3.3, U8 BTS50010-1TAD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

Commit message: Añade las celdas 6 y 7 (canales directos) y alarga la placa 47,7 mm
Hojas Celda6 y Celda7 en el esquemático con los canales idénticos a los demás;
los ESP32_OUT de las 9 salidas directas (canal 4 de la Celda5 y las celdas 6 y 7)
se amarran a +3,3 V en la raíz. En el PCB se alarga el contorno, los planos y las
tiras de +12 V; la Celda6 va en el frente como copia de la Celda3 y la Celda7 en B.Cu
colocada y ruteada con vías libres en todas las capas, con puentes en las islas del
plano +3,3 V. Quedan 3 conexiones sin rutear en la Celda7 y las uniones de +12 V
del reverso. Se documenta en CONTEXTO_PROYECTO.md.
Parts:
- added C501: 100uF 16V, Capacitor_SMD:CP_Elec_6.3x5.4, F.Cu at (-101.5, 240.1)
- added C502: 100nF, Capacitor_SMD:C_0805_2012Metric, F.Cu at (-96.0, 237.1)
- added C503: 1uF 25V, Capacitor_SMD:CP_Elec_4x5.4, F.Cu at (-102.6, 212.9)
- added C504: 100nF, Capacitor_SMD:C_0805_2012Metric, F.Cu at (-95.4, 227.2)
- added C505: 1uF 25V, Capacitor_SMD:CP_Elec_4x5.4, F.Cu at (-73.1, 217.8)
- added C516: 1uF 25V, Capacitor_SMD:CP_Elec_4x5.4, F.Cu at (-73.5, 236.0)
- added C517: 1uF 25V, Capacitor_SMD:CP_Elec_4x5.4, F.Cu at (-93.4, 212.9)
- added C518: 1uF 25V, Capacitor_SMD:CP_Elec_4x5.4, F.Cu at (-113.0, 237.4)
- added C519: 1uF 25V, Capacitor_SMD:CP_Elec_4x5.4, F.Cu at (-122.1, 237.4)
- added C520: 100nF, Capacitor_SMD:C_0805_2012Metric, F.Cu at (-115.7, 251.5)
- added C521: 1uF 25V, Capacitor_SMD:CP_Elec_4x5.4, F.Cu at (-144.0, 232.0)
- added C522: 1uF 25V, Capacitor_SMD:CP_Elec_4x5.4, F.Cu at (-143.8, 213.0)
- added C601: 100uF 16V, Capacitor_SMD:CP_Elec_6.3x5.4, B.Cu at (-116.5, 244.2)
- added C602: 100nF, Capacitor_SMD:C_0805_2012Metric, B.Cu at (-122.0, 242.5)
- added C603: 1uF 25V, Capacitor_SMD:CP_Elec_4x5.4, B.Cu at (-114.8, 217.6)
- added C604: 100nF, Capacitor_SMD:C_0805_2012Metric, B.Cu at (-120.7, 231.3)
- added C605: 1uF 25V, Capacitor_SMD:CP_Elec_4x5.4, B.Cu at (-144.3, 222.5)
- added C616: 1uF 25V, Capacitor_SMD:CP_Elec_4x5.4, B.Cu at (-143.7, 240.7)
- added C617: 1uF 25V, Capacitor_SMD:CP_Elec_4x5.4, B.Cu at (-125.0, 215.7)
- added C618: 1uF 25V, Capacitor_SMD:CP_Elec_4x5.4, B.Cu at (-107.4, 244.5)
- added C619: 1uF 25V, Capacitor_SMD:CP_Elec_4x5.4, B.Cu at (-94.5, 245.1)
- added C620: 100nF, Capacitor_SMD:C_0805_2012Metric, B.Cu at (-100.9, 256.3)
- added C621: 1uF 25V, Capacitor_SMD:CP_Elec_4x5.4, B.Cu at (-72.6, 236.7)
- added C622: 1uF 25V, Capacitor_SMD:CP_Elec_4x5.4, B.Cu at (-72.9, 217.7)
- added D501: BAT54C, Package_TO_SOT_SMD:SOT-23, F.Cu at (-83.9, 217.1)
- added D502: LED verde, LED_SMD:LED_0805_2012Metric, F.Cu at (-76.5, 212.0)
- added D503: LED rojo, LED_SMD:LED_0805_2012Metric, F.Cu at (-76.5, 214.3)
- added D507: LED verde, LED_SMD:LED_0805_2012Metric, F.Cu at (-77.2, 230.2)
- added D508: BAT54C, Package_TO_SOT_SMD:SOT-23, F.Cu at (-84.9, 235.2)
- added D509: LED rojo, LED_SMD:LED_0805_2012Metric, F.Cu at (-77.2, 232.5)
- added D510: LED rojo, LED_SMD:LED_0805_2012Metric, F.Cu at (-140.4, 235.4)
- added D511: LED rojo, LED_SMD:LED_0805_2012Metric, F.Cu at (-140.8, 217.7)
- added D512: LED verde, LED_SMD:LED_0805_2012Metric, F.Cu at (-140.4, 237.6)
- added D513: LED verde, LED_SMD:LED_0805_2012Metric, F.Cu at (-140.8, 220.0)
- added D514: BAT54C, Package_TO_SOT_SMD:SOT-23, F.Cu at (-133.1, 232.6)
- added D515: BAT54C, Package_TO_SOT_SMD:SOT-23, F.Cu at (-133.2, 215.2)
- added D601: BAT54C, Package_TO_SOT_SMD:SOT-23, B.Cu at (-133.8, 229.0)
- added D602: LED verde, LED_SMD:LED_0805_2012Metric, B.Cu at (-140.1, 216.7)
- added D603: LED rojo, LED_SMD:LED_0805_2012Metric, B.Cu at (-139.9, 219.0)
- added D607: LED verde, LED_SMD:LED_0805_2012Metric, B.Cu at (-139.5, 234.9)
- added D608: BAT54C, Package_TO_SOT_SMD:SOT-23, B.Cu at (-131.7, 239.9)
- added D609: LED rojo, LED_SMD:LED_0805_2012Metric, B.Cu at (-139.3, 237.2)
- added D610: LED rojo, LED_SMD:LED_0805_2012Metric, B.Cu at (-76.9, 240.1)
- added D611: LED rojo, LED_SMD:LED_0805_2012Metric, B.Cu at (-74.2, 222.7)
- added D612: LED verde, LED_SMD:LED_0805_2012Metric, B.Cu at (-75.6, 242.6)
- added D613: LED verde, LED_SMD:LED_0805_2012Metric, B.Cu at (-75.9, 224.9)
- added D614: BAT54C, Package_TO_SOT_SMD:SOT-23, B.Cu at (-83.5, 237.3)
- added D615: BAT54C, Package_TO_SOT_SMD:SOT-23, B.Cu at (-83.5, 219.9)
- added Q501: MMBT2222A, Package_TO_SOT_SMD:SOT-23, F.Cu at (-83.9, 212.1)
- added Q502: MMBT2222A, Package_TO_SOT_SMD:SOT-23, F.Cu at (-84.1, 220.8)
- added Q503: MMBT2222A, Package_TO_SOT_SMD:SOT-23, F.Cu at (-84.9, 230.2)
- added Q504: MMBT2222A, Package_TO_SOT_SMD:SOT-23, F.Cu at (-85.0, 239.2)
- added Q505: MMBT2222A, Package_TO_SOT_SMD:SOT-23, F.Cu at (-133.2, 228.6)
- added Q506: MMBT2222A, Package_TO_SOT_SMD:SOT-23, F.Cu at (-131.9, 211.2)
- added Q507: MMBT2222A, Package_TO_SOT_SMD:SOT-23, F.Cu at (-132.9, 237.6)
- added Q508: MMBT2222A, Package_TO_SOT_SMD:SOT-23, F.Cu at (-133.3, 220.0)
- added Q601: MMBT2222A, Package_TO_SOT_SMD:SOT-23, B.Cu at (-133.3, 217.9)
- added Q602: MMBT2222A, Package_TO_SOT_SMD:SOT-23, B.Cu at (-137.9, 229.5)
- added Q603: MMBT2222A, Package_TO_SOT_SMD:SOT-23, B.Cu at (-131.7, 234.6)
- added Q604: MMBT2222A, Package_TO_SOT_SMD:SOT-23, B.Cu at (-131.6, 243.9)
- added Q605: MMBT2222A, Package_TO_SOT_SMD:SOT-23, B.Cu at (-84.0, 233.3)
- added Q606: MMBT2222A, Package_TO_SOT_SMD:SOT-23, B.Cu at (-84.7, 215.8)
- added Q607: MMBT2222A, Package_TO_SOT_SMD:SOT-23, B.Cu at (-83.7, 242.3)
- added Q608: MMBT2222A, Package_TO_SOT_SMD:SOT-23, B.Cu at (-83.4, 224.7)
- added R501: umbral, Resistor_THT:R_Axial_DIN0207_L6.3mm_D2.5mm_P10.16mm_Horizontal, F.Cu at (-123.1, 225.8)
- added R502: 10k, Resistor_SMD:R_0805_2012Metric, F.Cu at (-113.4, 228.3)
- added R503: 10k, Resistor_SMD:R_0805_2012Metric, F.Cu at (-108.3, 222.4)
- added R504: 4.7k, Resistor_SMD:R_0805_2012Metric, F.Cu at (-87.7, 217.8)
- added R505: 4.7k, Resistor_SMD:R_0805_2012Metric, F.Cu at (-87.7, 215.8)
- added R506: 10k, Resistor_SMD:R_0805_2012Metric, F.Cu at (-99.1, 212.2)
- added R507: 100k, Resistor_SMD:R_0805_2012Metric, F.Cu at (-87.7, 211.6)
- added R508: 100k, Resistor_SMD:R_0805_2012Metric, F.Cu at (-80.9, 218.6)
- added R509: 1k, Resistor_SMD:R_0805_2012Metric, F.Cu at (-76.6, 218.6)
- added R510: 2.2k, Resistor_SMD:R_0805_2012Metric, F.Cu at (-80.2, 212.1)
- added R511: 4.7k, Resistor_SMD:R_0805_2012Metric, F.Cu at (-88.0, 219.8)
- added R512: 1k, Resistor_SMD:R_0805_2012Metric, F.Cu at (-80.0, 214.3)
- added R519: 4.7k, Resistor_SMD:R_0805_2012Metric, F.Cu at (-88.7, 236.2)
- added R520: 4.7k, Resistor_SMD:R_0805_2012Metric, F.Cu at (-88.7, 234.0)
- added R521: 2.2k, Resistor_SMD:R_0805_2012Metric, F.Cu at (-80.9, 230.2)
- added R522: 100k, Resistor_SMD:R_0805_2012Metric, F.Cu at (-88.8, 229.8)
- added R523: 100k, Resistor_SMD:R_0805_2012Metric, F.Cu at (-81.7, 236.8)
- added R524: 1k, Resistor_SMD:R_0805_2012Metric, F.Cu at (-77.2, 236.7)
- added R525: 1k, Resistor_SMD:R_0805_2012Metric, F.Cu at (-81.0, 232.5)
- added R526: 4.7k, Resistor_SMD:R_0805_2012Metric, F.Cu at (-88.7, 238.2)
- added R527: 10k, Resistor_SMD:R_0805_2012Metric, F.Cu at (-106.3, 222.4)
- added R528: 10k, Resistor_SMD:R_0805_2012Metric, F.Cu at (-96.9, 212.2)
- added R529: umbral, Resistor_THT:R_Axial_DIN0207_L6.3mm_D2.5mm_P10.16mm_Horizontal, F.Cu at (-123.0, 210.3)
- added R530: 10k, Resistor_SMD:R_0805_2012Metric, F.Cu at (-113.5, 212.8)
- added R531: 10k, Resistor_SMD:R_0805_2012Metric, F.Cu at (-116.5, 236.7)
- added R532: 10k, Resistor_SMD:R_0805_2012Metric, F.Cu at (-118.5, 236.7)
- added R533: 1k, Resistor_SMD:R_0805_2012Metric, F.Cu at (-136.9, 235.4)
- added R534: 1k, Resistor_SMD:R_0805_2012Metric, F.Cu at (-137.2, 217.7)
- added R535: 4.7k, Resistor_SMD:R_0805_2012Metric, F.Cu at (-129.2, 229.7)
- added R536: 4.7k, Resistor_SMD:R_0805_2012Metric, F.Cu at (-128.1, 212.2)
- added R537: 4.7k, Resistor_SMD:R_0805_2012Metric, F.Cu at (-129.2, 231.6)
- added R538: 4.7k, Resistor_SMD:R_0805_2012Metric, F.Cu at (-129.2, 233.6)
- added R539: 4.7k, Resistor_SMD:R_0805_2012Metric, F.Cu at (-129.4, 214.2)
- added R540: 4.7k, Resistor_SMD:R_0805_2012Metric, F.Cu at (-129.4, 216.2)
- added R541: 2.2k, Resistor_SMD:R_0805_2012Metric, F.Cu at (-136.9, 237.6)
- added R542: 2.2k, Resistor_SMD:R_0805_2012Metric, F.Cu at (-137.1, 220.0)
- added R543: 100k, Resistor_SMD:R_0805_2012Metric, F.Cu at (-128.9, 238.1)
- added R544: 100k, Resistor_SMD:R_0805_2012Metric, F.Cu at (-136.4, 231.2)
- added R545: 100k, Resistor_SMD:R_0805_2012Metric, F.Cu at (-129.3, 220.7)
- added R546: 100k, Resistor_SMD:R_0805_2012Metric, F.Cu at (-135.3, 212.5)
- added R547: 1k, Resistor_SMD:R_0805_2012Metric, F.Cu at (-140.5, 231.2)
- added R548: 1k, Resistor_SMD:R_0805_2012Metric, F.Cu at (-140.3, 212.3)
- added R549: umbral, Resistor_THT:R_Axial_DIN0207_L6.3mm_D2.5mm_P10.16mm_Horizontal, F.Cu at (-123.0, 215.7)
- added R550: 10k, Resistor_SMD:R_0805_2012Metric, F.Cu at (-113.4, 218.1)
- added R551: umbral, Resistor_THT:R_Axial_DIN0207_L6.3mm_D2.5mm_P10.16mm_Horizontal, F.Cu at (-123.0, 220.7)
- added R552: 10k, Resistor_SMD:R_0805_2012Metric, F.Cu at (-113.4, 223.3)
- added R553: 10k, Resistor_SMD:R_0805_2012Metric, F.Cu at (-104.3, 222.4)
- added R554: 10k, Resistor_SMD:R_0805_2012Metric, F.Cu at (-102.3, 222.4)
- added R601: umbral, Resistor_THT:R_Axial_DIN0207_L6.3mm_D2.5mm_P10.16mm_Horizontal, B.Cu at (-89.5, 240.0)
- added R602: 10k, Resistor_SMD:R_0805_2012Metric, B.Cu at (-106.3, 230.5)
- added R603: 10k, Resistor_SMD:R_0805_2012Metric, B.Cu at (-108.4, 227.1)
- added R604: 4.7k, Resistor_SMD:R_0805_2012Metric, B.Cu at (-129.9, 228.1)
- added R605: 4.7k, Resistor_SMD:R_0805_2012Metric, B.Cu at (-131.9, 215.0)
- added R606: 10k, Resistor_SMD:R_0805_2012Metric, B.Cu at (-118.5, 213.2)
- added R607: 100k, Resistor_SMD:R_0805_2012Metric, B.Cu at (-129.8, 212.8)
- added R608: 100k, Resistor_SMD:R_0805_2012Metric, B.Cu at (-136.2, 223.2)
- added R609: 1k, Resistor_SMD:R_0805_2012Metric, B.Cu at (-140.0, 223.3)
- added R610: 2.2k, Resistor_SMD:R_0805_2012Metric, B.Cu at (-136.5, 214.9)
- added R611: 4.7k, Resistor_SMD:R_0805_2012Metric, B.Cu at (-128.2, 223.8)
- added R612: 1k, Resistor_SMD:R_0805_2012Metric, B.Cu at (-137.0, 226.1)
- added R619: 4.7k, Resistor_SMD:R_0805_2012Metric, B.Cu at (-127.8, 240.9)
- added R620: 4.7k, Resistor_SMD:R_0805_2012Metric, B.Cu at (-127.8, 238.7)
- added R621: 2.2k, Resistor_SMD:R_0805_2012Metric, B.Cu at (-135.7, 234.2)
- added R622: 100k, Resistor_SMD:R_0805_2012Metric, B.Cu at (-127.8, 234.4)
- added R623: 100k, Resistor_SMD:R_0805_2012Metric, B.Cu at (-134.9, 241.4)
- added R624: 1k, Resistor_SMD:R_0805_2012Metric, B.Cu at (-139.5, 241.3)
- added R625: 1k, Resistor_SMD:R_0805_2012Metric, B.Cu at (-135.7, 237.2)
- added R626: 4.7k, Resistor_SMD:R_0805_2012Metric, B.Cu at (-127.8, 243.1)
- added R627: 10k, Resistor_SMD:R_0805_2012Metric, B.Cu at (-113.0, 229.9)
- added R628: 10k, Resistor_SMD:R_0805_2012Metric, B.Cu at (-119.8, 216.8)
- added R629: umbral, Resistor_THT:R_Axial_DIN0207_L6.3mm_D2.5mm_P10.16mm_Horizontal, B.Cu at (-95.2, 215.0)
- added R630: 10k, Resistor_SMD:R_0805_2012Metric, B.Cu at (-104.6, 219.7)
- added R631: 10k, Resistor_SMD:R_0805_2012Metric, B.Cu at (-101.4, 243.5)
- added R632: 10k, Resistor_SMD:R_0805_2012Metric, B.Cu at (-98.2, 243.5)
- added R633: 1k, Resistor_SMD:R_0805_2012Metric, B.Cu at (-79.7, 244.5)
- added R634: 1k, Resistor_SMD:R_0805_2012Metric, B.Cu at (-78.7, 220.9)
- added R635: 4.7k, Resistor_SMD:R_0805_2012Metric, B.Cu at (-87.8, 234.3)
- added R636: 4.7k, Resistor_SMD:R_0805_2012Metric, B.Cu at (-90.8, 217.0)
- added R637: 4.7k, Resistor_SMD:R_0805_2012Metric, B.Cu at (-87.5, 236.5)
- added R638: 4.7k, Resistor_SMD:R_0805_2012Metric, B.Cu at (-91.1, 237.0)
- added R639: 4.7k, Resistor_SMD:R_0805_2012Metric, B.Cu at (-91.2, 219.2)
- added R640: 4.7k, Resistor_SMD:R_0805_2012Metric, B.Cu at (-87.3, 220.3)
- added R641: 2.2k, Resistor_SMD:R_0805_2012Metric, B.Cu at (-79.7, 242.3)
- added R642: 2.2k, Resistor_SMD:R_0805_2012Metric, B.Cu at (-79.5, 225.3)
- added R643: 100k, Resistor_SMD:R_0805_2012Metric, B.Cu at (-87.7, 242.8)
- added R644: 100k, Resistor_SMD:R_0805_2012Metric, B.Cu at (-80.2, 235.9)
- added R645: 100k, Resistor_SMD:R_0805_2012Metric, B.Cu at (-86.8, 227.6)
- added R646: 100k, Resistor_SMD:R_0805_2012Metric, B.Cu at (-81.1, 216.3)
- added R647: 1k, Resistor_SMD:R_0805_2012Metric, B.Cu at (-76.2, 235.9)
- added R648: 1k, Resistor_SMD:R_0805_2012Metric, B.Cu at (-76.5, 217.0)
- added R649: umbral, Resistor_THT:R_Axial_DIN0207_L6.3mm_D2.5mm_P10.16mm_Horizontal, B.Cu at (-101.0, 208.4)
- added R650: 10k, Resistor_SMD:R_0805_2012Metric, B.Cu at (-103.2, 222.8)
- added R651: umbral, Resistor_THT:R_Axial_DIN0207_L6.3mm_D2.5mm_P10.16mm_Horizontal, B.Cu at (-89.7, 225.4)
- added R652: 10k, Resistor_SMD:R_0805_2012Metric, B.Cu at (-103.2, 228.0)
- added R653: 10k, Resistor_SMD:R_0805_2012Metric, B.Cu at (-110.8, 227.1)
- added R654: 10k, Resistor_SMD:R_0805_2012Metric, B.Cu at (-114.8, 226.3)
- added U501: LM339D, Package_SO:SOIC-14_3.9x8.7mm_P1.27mm, F.Cu at (-105.3, 230.4)
- added U502: 74HC132D, Package_SO:SOIC-14_3.9x8.7mm_P1.27mm, F.Cu at (-95.4, 221.4)
- added U503: BTS50010-1TAD, Package_TO_SOT_SMD:TO-263-7_TabPin4, F.Cu at (-62.4, 216.1)
- added U508: BTS50010-1TAD, Package_TO_SOT_SMD:TO-263-7_TabPin4, F.Cu at (-62.4, 234.8)
- added U509: 74HC132D, Package_SO:SOIC-14_3.9x8.7mm_P1.27mm, F.Cu at (-115.7, 245.8)
- added U510: BTS50010-1TAD, Package_TO_SOT_SMD:TO-263-7_TabPin4, F.Cu at (-154.7, 232.9)
- added U511: BTS50010-1TAD, Package_TO_SOT_SMD:TO-263-7_TabPin4, F.Cu at (-154.7, 216.1)
- added U601: LM339D, Package_SO:SOIC-14_3.9x8.7mm_P1.27mm, B.Cu at (-105.3, 236.3)
- added U602: 74HC132D, Package_SO:SOIC-14_3.9x8.7mm_P1.27mm, B.Cu at (-122.6, 223.9)
- added U603: BTS50010-1TAD, Package_TO_SOT_SMD:TO-263-7_TabPin4, B.Cu at (-154.3, 220.8)
- added U608: BTS50010-1TAD, Package_TO_SOT_SMD:TO-263-7_TabPin4, B.Cu at (-154.3, 239.5)
- added U609: 74HC132D, Package_SO:SOIC-14_3.9x8.7mm_P1.27mm, B.Cu at (-101.0, 250.5)
- added U610: BTS50010-1TAD, Package_TO_SOT_SMD:TO-263-7_TabPin4, B.Cu at (-62.3, 234.6)
- added U611: BTS50010-1TAD, Package_TO_SOT_SMD:TO-263-7_TabPin4, B.Cu at (-62.0, 215.8)
Connections:
- R440 pad 2: /Celda5/ESP32_OUT4 -> +3.3V
Routing:
- net +3.3V: track 403.0 -> 541.5 mm, vias 112 -> 165
- net GND: track 382.1 -> 515.7 mm, vias 201 -> 273
- net +12V: track 431.6 -> 527.0 mm
- net Net-(U501C--): track 0.00 -> 95.3 mm, vias 0 -> 7
- net Net-(U501A--): track 0.00 -> 88.7 mm, vias 0 -> 3
- net Net-(U601A--): track 0.00 -> 86.6 mm, vias 0 -> 8
- net Net-(U501B--): track 0.00 -> 86.4 mm, vias 0 -> 3
- net Net-(U601D--): track 0.00 -> 76.0 mm, vias 0 -> 4
- net Net-(U501D--): track 0.00 -> 75.6 mm, vias 0 -> 4
- net Net-(U601B--): track 0.00 -> 67.2 mm, vias 0 -> 4
- net /Celda7/FALLA4: track 0.00 -> 62.7 mm, vias 0 -> 2
- net Net-(U601C--): track 0.00 -> 59.3 mm, vias 0 -> 6
- net Net-(Q506-C): track 0.00 -> 56.8 mm, vias 0 -> 2
- net Net-(Q505-C): track 0.00 -> 55.8 mm, vias 0 -> 2
- net Net-(Q504-C): track 0.00 -> 55.6 mm, vias 0 -> 2
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Other:
- board size 123 x 191.1 mm -> 123 x 238.8 mm

Commit message: Actualiza la PCB con los ajustes hechos en KiCad tras las celdas 6 y 7
Cambios manuales del usuario sobre la placa alargada y ruta de salida de
Gerber guardada en el proyecto.
Parts:
- moved J2 238.6 mm to (-163.0, 73.0), turned to 90 degrees
- moved J1 223.2 mm to (-163.0, 90.0), turned to 90 degrees
- moved C6 79.5 mm to (-80.0, 105.0)
Changed lines of the file:
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@@
 	(footprint "Capacitor_SMD:C_0805_2012Metric"
 		(layer "F.Cu")
-		(at -2.35 122)
+		(at -80 105)
 		(descr "Capacitor SMD 0805 (2012 Metric), square (rectangular) end terminal, IPC-7351 nominal, (Body size source: IPC-SM-782 page 76, https://www.pcb-3d.com/wordpress/wp-content/uploads/ipc-sm-782a_amendment_1_and_2.pdf, https://docs.google.com/spreadsheets/d/1BsfQQcO9C6DZCsRaXUlFlo91Tg2WpOkGARC1WS5S8t0/edit?usp=sharing)")
 		(tags "capacitor")
@@
 	(footprint "MountingHole:MountingHole_6.4mm_M6_Pad"
 		(layer "F.Cu")
-		(at 58.25 60.5)
+		(at -163 90 90)
 		(descr "Mounting Hole 6.4mm, M6, generated by kicad-footprint-generator mountinghole.py")
 		(tags "mountinghole M6")
 		(property "Reference" "J1"
-			(at 0 -7.35 0)
+			(at 0 -7.35 90)
 			(layer "F.SilkS")
 			(effects
@@
 		)
 		(property "Value" "+12V borne M6"
-			(at 0 7.35 0)
+			(at 0 7.35 90)
 			(layer "F.Fab")
 			(effects
@@
 		)
 		(property "Datasheet" ""
-			(at 0 0 0)
+			(at 0 0 90)
 			(layer "F.Fab")
 			(hide yes)
@@
 		)
 		(property "Description" "Generic screw terminal, single row, 01x01, script generated (kicad-library-utils/schlib/autogen/connector/)"
-			(at 0 0 0)
+			(at 0 0 90)
 			(layer "F.Fab")
 			(hide yes)
@@
 		)
 		(property "KiLib_Generator" "mounting_hardware/mounting_hole"
-			(at 0 0 0)
+			(at 0 0 90)
 			(layer "F.SilkS")
 			(hide yes)
@@
 		)
 		(fp_text user "${REFERENCE}"
-			(at 0 0 0)
+			(at 0 0 90)
 			(layer "F.Fab")
 			(effects
@@
 		)
 		(pad "1" thru_hole circle
-			(at 0 0)
+			(at 0 0 90)
 			(size 12.8 12.8)
 			(drill 6.4)
@@
 	(footprint "MountingHole:MountingHole_5.3mm_M5_Pad"
 		(layer "F.Cu")
-		(at 75.25 60.5)
+		(at -163 73 90)
 		(descr "Mounting Hole 5.3mm, M5, generated by kicad-footprint-generator mountinghole.py")
 		(tags "mountinghole M5")
 		(property "Reference" "J2"
-			(at 0 -6.25 0)
+			(at 0 -6.25 90)
 			(layer "F.SilkS")
 			(effects
@@
 		)
 		(property "Value" "GND borne M5"
-			(at 0 6.25 0)
+			(at 0 6.25 90)
 			(layer "F.Fab")
 			(effects
@@
 		)
 		(property "Datasheet" ""
-			(at 0 0 0)
+			(at 0 0 90)
 			(layer "F.Fab")
 			(hide yes)
@@
 		)
 		(property "Description" "Generic screw terminal, single row, 01x01, script generated (kicad-library-utils/schlib/autogen/connector/)"
-			(at 0 0 0)
+			(at 0 0 90)
 			(layer "F.Fab")
 			(hide yes)
@@
 		)
 		(property "KiLib_Generator" "mounting_hardware/mounting_hole"
-			(at 0 0 0)
+			(at 0 0 90)
 			(layer "F.SilkS")
 			(hide yes)
@@
 		)
 		(fp_text user "${REFERENCE}"
-			(at 0 0 0)
+			(at 0 0 90)
 			(layer "F.Fab")
 			(effects
@@
 		)
 		(pad "1" thru_hole circle
-			(at 0 0)
+			(at 0 0 90)
 			(size 10.6 10.6)
 			(drill 5.3)
