File: placa-slave/placa-slave.kicad_sch (KiCad schematic)
At the start: 27 parts, among them J1 +12V borne M6, J10 Enlace_placas, J2 GND borne M5, U5 MCP23017-E/SO, U6 LM5164DDA, U7 AP2112K-3.3

Commit message: Cablea alimentación e I2C de las placas y replica las celdas en los PCB
Esquemáticos raíz: se cablean VDD, VSS, RESET, direcciones y SDA/SCL de los
MCP, los pull-ups de I2C (solo en la master), el LDO de 3,3 V y la entrada de
+12 V de la master, y la unión de las redes del bloque de poder en la slave.

PCB: nuevo herramientas/replicar_celdas_pcb.py que copia la celda dorada por
traslación en cada placa (master en una fila de 3 celdas, slave en 2 x 2), con
pistas, vías, serigrafía y planos GND/+3,3 V. Coloca además las huellas de la
raíz (ESP32, MCP, bloque de poder, conector) en una franja provisional bajo
las celdas, ya enlazadas al esquemático. Sin tiras de +12 V a propósito: se
dibujan al final. La master incluye los ajustes manuales hechos en KiCad.
Parts:
- removed D6: Schottky 1A (SS14), Diode_SMD:D_SMA, symbol Device:D_Schottky
Connections:
- net V3V3_OUT is gone; now on net +3.3V: C15.1, U7.5 (VOUT)
- net +3.3V: now also C6.1, U5.15 (A0), U5.18 (~{RESET}), U5.9 (V_{DD})
- net GND: now also C6.2, U5.10 (V_{SS}), U5.16 (A1), U5.17 (A2)
- net LINK_5V: now also C11.1, C12.2, C14.1, L1.2, R13.1, U7.1 (VIN), U7.3 (EN)
- net SCL: now also U5.12 (SCK)
- net SDA: now also U5.13 (SDA)
- net VBB renamed +12V
- no-connect marks 1 -> 4
